File: pcb-source/file5D66FCEB.kicad_sch (KiCad schematic)
At the start: 13 parts, among them J5 Conn_01x02_Female, U10 AMS1117-3.3, U3 AZ1117-5.0, U7 AMS1117-3.3, U8 AMS1117-1.8

Commit message: Working RTC with USART2 as SPI master
Changed lines of the file:
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@@
 (kicad_sch
-	(version 20231120)
+	(version 20250114)
 	(generator "eeschema")
-	(generator_version "8.0")
+	(generator_version "9.0")
 	(paper "A4")
 	(title_block
@@
 		)
 		(instances
-			(project ""
+			(project "AtariHDisk4"
 				(path "/b85bd53e-a419-4638-ac5c-9132c68f9083/00000000-0000-0000-0000-00005d66fcec"
 					(reference "R6")
