File: pcb-source/file5D6A3596.kicad_sch (KiCad schematic)
At the start: 21 parts, among them J2 Program_enable, J6 Conn_02x03_Odd_Even, J7 ST-LINK, U2 MAX3232, U5 MCP795xx, U6 STM32C031CxT, Y1 32KHz

Commit message: Working RTC with USART2 as SPI master
Parts:
- C10, C2, C22, C7: value C -> 0.1uF 50V
- C29, C30: value 3pF -> 10pF
Other:
- moved on the sheet: C21
